File: hardware/mainboard/currentsensor.kicad_sch (KiCad schematic)
At the start: 9 parts, among them U5 ACS759, U6 ACS712

Commit message: Mainboard routeado.
Parts:
- renumbered JP2 to JP1
Changed lines of the file:
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@@
   (symbol (lib_id "power:GND") (at 130.81 137.16 0) (unit 1)
     (in_bom yes) (on_board yes)
-    (property "Reference" "#PWR055" (id 0) (at 130.81 143.51 0)
+    (property "Reference" "#PWR054" (id 0) (at 130.81 143.51 0)
       (effects (font (size 1.27 1.27)) hide)
     )
@@
   (symbol (lib_id "power:GND") (at 142.24 137.16 0) (unit 1)
     (in_bom yes) (on_board yes)
-    (property "Reference" "#PWR057" (id 0) (at 142.24 143.51 0)
+    (property "Reference" "#PWR056" (id 0) (at 142.24 143.51 0)
       (effects (font (size 1.27 1.27)) hide)
     )
@@
   (symbol (lib_id "power:GND") (at 162.56 137.16 0) (mirror y) (unit 1)
     (in_bom yes) (on_board yes)
-    (property "Reference" "#PWR059" (id 0) (at 162.56 143.51 0)
+    (property "Reference" "#PWR058" (id 0) (at 162.56 143.51 0)
       (effects (font (size 1.27 1.27)) hide)
     )
@@
   (symbol (lib_id "power:+3V3") (at 130.81 110.49 0) (unit 1)
     (in_bom yes) (on_board yes)
-    (property "Reference" "#PWR054" (id 0) (at 130.81 114.3 0)
+    (property "Reference" "#PWR053" (id 0) (at 130.81 114.3 0)
       (effects (font (size 1.27 1.27)) hide)
     )
@@
   (symbol (lib_id "power:+5V") (at 165.1 63.5 0) (unit 1)
     (in_bom yes) (on_board yes)
-    (property "Reference" "#PWR060" (id 0) (at 165.1 67.31 0)
+    (property "Reference" "#PWR059" (id 0) (at 165.1 67.31 0)
       (effects (font (size 1.27 1.27)) hide)
     )
@@
   (symbol (lib_id "power:GND") (at 165.1 92.71 0) (unit 1)
     (in_bom yes) (on_board yes)
-    (property "Reference" "#PWR061" (id 0) (at 165.1 99.06 0)
+    (property "Reference" "#PWR060" (id 0) (at 165.1 99.06 0)
       (effects (font (size 1.27 1.27)) hide)
     )
@@
   (symbol (lib_id "power:GND") (at 148.59 92.71 0) (unit 1)
     (in_bom yes) (on_board yes)
-    (property "Reference" "#PWR058" (id 0) (at 148.59 99.06 0)
+    (property "Reference" "#PWR057" (id 0) (at 148.59 99.06 0)
       (effects (font (size 1.27 1.27)) hide)
     )
@@
   (symbol (lib_id "power:GND") (at 137.16 92.71 0) (unit 1)
     (in_bom yes) (on_board yes)
-    (property "Reference" "#PWR056" (id 0) (at 137.16 99.06 0)
+    (property "Reference" "#PWR055" (id 0) (at 137.16 99.06 0)
       (effects (font (size 1.27 1.27)) hide)
     )
@@
   (symbol (lib_id "power:GND") (at 121.92 92.71 0) (unit 1)
     (in_bom yes) (on_board yes)
-    (property "Reference" "#PWR053" (id 0) (at 121.92 99.06 0)
+    (property "Reference" "#PWR052" (id 0) (at 121.92 99.06 0)
       (effects (font (size 1.27 1.27)) hide)
     )
@@
   (symbol (lib_id "kicad-rescue:SolderJumper_3_Bridged12-Jumper") (at 106.68 107.95 270) (mirror x) (unit 1)
     (in_bom yes) (on_board yes)
-    (property "Reference" "JP2" (id 0) (at 108.4072 107.95 90)
-      (effects (font (size 1.27 1.27)) (justify left))
-    )
+    (property "Reference" "JP1" (id 0) (at 108.4072 107.95 90)
+      (effects (font (size 1.27 1.27)) (justify left))
+    )
