File: hardware/mainboard/io.kicad_sch (KiCad schematic)
At the start: 3 parts, among them J10 Conn_01x10, J11 Conn_01x06

Commit message: Mainboard routeado.
Parts:
- renumbered JP3 to JP2
Changed lines of the file:
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@@
   (symbol (lib_id "Jumper:SolderJumper_2_Open") (at 163.83 104.14 90) (unit 1)
     (in_bom yes) (on_board yes)
-    (property "Reference" "JP3" (id 0) (at 166.37 102.87 0)
+    (property "Reference" "JP2" (id 0) (at 166.37 102.87 0)
       (effects (font (size 1.27 1.27)) (justify right))
     )
@@
   (symbol (lib_id "power:+12V") (at 163.83 96.52 0) (unit 1)
     (in_bom yes) (on_board yes)
-    (property "Reference" "#PWR067" (id 0) (at 163.83 100.33 0)
+    (property "Reference" "#PWR066" (id 0) (at 163.83 100.33 0)
       (effects (font (size 1.27 1.27)) hide)
     )
@@
   (symbol (lib_id "power:GND") (at 184.15 106.68 0) (unit 1)
     (in_bom yes) (on_board yes)
-    (property "Reference" "#PWR?" (id 0) (at 184.15 113.03 0)
+    (property "Reference" "#PWR067" (id 0) (at 184.15 113.03 0)
       (effects (font (size 1.27 1.27)) hide)
     )
