File: hardware/mainboard/psu.kicad_sch (KiCad schematic)
At the start: 9 parts, among them U3 LM2596S-3.3, U4 AMS1117-5.0

Commit message: Mainboard routeado.
Parts:
- renumbered R17 to R18
Changed lines of the file:
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@@
   (symbol (lib_id "Device:R") (at 54.61 99.06 0) (unit 1)
     (in_bom yes) (on_board yes)
-    (property "Reference" "R17" (id 0) (at 56.388 97.8916 0)
+    (property "Reference" "R18" (id 0) (at 56.388 97.8916 0)
       (effects (font (size 1.27 1.27)) (justify left))
     )
@@
   (symbol (lib_id "power:GND") (at 179.07 104.14 0) (unit 1)
     (in_bom yes) (on_board yes)
-    (property "Reference" "#PWR050" (id 0) (at 179.07 110.49 0)
+    (property "Reference" "#PWR049" (id 0) (at 179.07 110.49 0)
       (effects (font (size 1.27 1.27)) hide)
     )
